File: version2/tcsmonitor-pcb/tcsmonitor-pcb.kicad_pcb (KiCad board)
At the start: 2 copper layers, 11 parts, among them J1 Screw_Terminal_01x02, Q1 Q_NPN_BCE, U1 WeMos_D1_mini, X1 Arduino_Pro_Mini

Commit message: bak-Dateien gelöscht. Connectoren eingefügt.
Parts:
- added J1_A1: Conn_01x04_Female, Connector_PinHeader_2.54mm:PinHeader_1x04_P2.54mm_Vertical, F.Cu at (193.0, 34.3)
- added J1_B1: Conn_01x04_Female, Connector_PinHeader_2.54mm:PinHeader_1x04_P2.54mm_Vertical, F.Cu at (205.7, 34.3)
- added J_USB1: Conn_01x05_Male, Connector_PinHeader_2.54mm:PinHeader_1x05_P2.54mm_Vertical, F.Cu at (207.0, 95.2)
- J1: moved to F.Cu
- R1, R3: moved to B.Cu
- moved R3 72.7 mm to (114.3, 97.8), turned to 90 degrees
- moved R1 56.7 mm to (124.5, 90.2), turned to 270 degrees
- moved R6 26.9 mm to (85.1, 67.3)
- moved R4 26.2 mm to (109.2, 44.5)
- moved Q1 22.6 mm to (120.7, 43.2)
- moved R2 21.8 mm to (120.7, 58.4)
- moved R5 21.6 mm to (109.2, 38.1)
- moved U1 19.4 mm to (217.2, 58.4)
- moved R7 15.5 mm to (90.2, 45.7), turned to 90 degrees
- turned J1 to 270 degrees
Connections:
- U1 pad 10: Net-(U1-Pad10) -> GND
- U1 pad 9: Net-(U1-Pad9) -> VCC
- X1 pad 2A: Net-(X1-Pad2A) -> GND
- X1 pad 4A: Net-(X1-Pad4A) -> VCC
- X1 pad 4D: Net-(X1-Pad4D) -> GND
