File: version2/tcsmonitor-pcb/tcsmonitor-pcb.sch (KiCad schematic (older format))
At the start: 11 parts, among them J1 Screw_Terminal_01x02, Q1 Q_NPN_BCE, U1 WeMos_D1_mini, X1 Arduino_Pro_Mini

Commit message: minor changes
Connections:
- net GND: now also X1.2A (GND), X1.4D (Gnd)
- net VCC: now also X1.4A (Vcc)
Changed lines of the file:
@@
 Wire Wire Line
 	4900 3550 5000 3550
+$Comp
+L power:VCC #PWR0101
+U 1 1 5E2DC3EB
+P 6650 2850
+F 0 "#PWR0101" H 6650 2700 50  0001 C CNN
+F 1 "VCC" H 6667 3023 50  0000 C CNN
+F 2 "" H 6650 2850 50  0001 C CNN
+F 3 "" H 6650 2850 50  0001 C CNN
+	1    6650 2850
+	0    1    1    0
+$EndComp
+Wire Wire Line
+	6100 2850 6650 2850
+$Comp
+L power:GND #PWR0102
+U 1 1 5E2E7F6C
+P 6650 2650
+F 0 "#PWR0102" H 6650 2400 50  0001 C CNN
+F 1 "GND" H 6655 2477 50  0000 C CNN
+F 2 "" H 6650 2650 50  0001 C CNN
+F 3 "" H 6650 2650 50  0001 C CNN
+	1    6650 2650
+	0    -1   1    0
+$EndComp
+Wire Wire Line
+	6100 2650 6650 2650
+$Comp
+L power:GND #PWR0103
+U 1 1 5E2EBF84
+P 4650 2950
+F 0 "#PWR0103" H 4650 2700 50  0001 C CNN
+F 1 "GND" H 4655 2777 50  0000 C CNN
+F 2 "" H 4650 2950 50  0001 C CNN
+F 3 "" H 4650 2950 50  0001 C CNN
+	1    4650 2950
+	0    1    1    0
+$EndComp
+Wire Wire Line
+	4650 2950 5000 2950
 $EndSCHEMATC

Commit message: bak-Dateien gelöscht. Connectoren eingefügt.
Parts:
- added J1_A1, J1_B1: Conn_01x04_Female, Connector_PinHeader_2.54mm:PinHeader_1x04_P2.54mm_Vertical, symbol Connector:Conn_01x04_Female
- added J_USB1: Conn_01x05_Male, Connector_PinHeader_2.54mm:PinHeader_1x05_P2.54mm_Vertical, symbol Connector:Conn_01x05_Male
Connections:
- net GND: now also U1.10 (GND), J1_A1.4 (Pin_4), J1_B1.4 (Pin_4), J_USB1.5 (Pin_5)
- net VCC: now also U1.9 (5V), J1_A1.1 (Pin_1), J_USB1.1 (Pin_1)
- net at U1.15 (RX): now also J1_B1.2 (Pin_2)
- net at U1.16 (TX): now also J1_B1.3 (Pin_3)
- net at U1.8 (3V3): now also J1_B1.1 (Pin_1)
- net at X1.1D (1(Tx)): now also J1_A1.2 (Pin_2)
- net at X1.2D (0(Rx)): now also J1_A1.3 (Pin_3)
Changed lines of the file:
@@
 L power:VCC #PWR0101
 U 1 1 5E2DC3EB
-P 6650 2850
-F 0 "#PWR0101" H 6650 2700 50  0001 C CNN
-F 1 "VCC" H 6667 3023 50  0000 C CNN
-F 2 "" H 6650 2850 50  0001 C CNN
-F 3 "" H 6650 2850 50  0001 C CNN
-	1    6650 2850
+P 6350 2850
+F 0 "#PWR0101" H 6350 2700 50  0001 C CNN
+F 1 "VCC" H 6367 3023 50  0000 C CNN
+F 2 "" H 6350 2850 50  0001 C CNN
+F 3 "" H 6350 2850 50  0001 C CNN
+	1    6350 2850
 	0    1    1    0
 $EndComp
 Wire Wire Line
-	6100 2850 6650 2850
+	6100 2850 6350 2850
 $Comp
 L power:GND #PWR0102
 U 1 1 5E2E7F6C
-P 6650 2650
-F 0 "#PWR0102" H 6650 2400 50  0001 C CNN
-F 1 "GND" H 6655 2477 50  0000 C CNN
-F 2 "" H 6650 2650 50  0001 C CNN
-F 3 "" H 6650 2650 50  0001 C CNN
-	1    6650 2650
+P 6350 2650
+F 0 "#PWR0102" H 6350 2400 50  0001 C CNN
+F 1 "GND" H 6355 2477 50  0000 C CNN
+F 2 "" H 6350 2650 50  0001 C CNN
+F 3 "" H 6350 2650 50  0001 C CNN
+	1    6350 2650
 	0    -1   1    0
 $EndComp
 Wire Wire Line
-	6100 2650 6650 2650
+	6100 2650 6350 2650
 $Comp
 L power:GND #PWR0103
@@
 Wire Wire Line
 	4650 2950 5000 2950
+$Comp
+L Connector:Conn_01x04_Female J1_A1
+U 1 1 5E361570
+P 7400 1600
+F 0 "J1_A1" H 7428 1576 50  0000 L CNN
+F 1 "Conn_01x04_Female" H 7428 1485 50  0000 L CNN
+F 2 "Connector_PinHeader_2.54mm:PinHeader_1x04_P2.54mm_Vertical" H 7400 1600 50  0001 C CNN
+F 3 "~" H 7400 1600 50  0001 C CNN
+	1    7400 1600
+	1    0    0    -1
+$EndComp
+$Comp
+L Connector:Conn_01x04_Female J1_B1
+U 1 1 5E3646F9
+P 8500 1600
+F 0 "J1_B1" H 8392 1885 50  0000 C CNN
+F 1 "Conn_01x04_Female" H 8392 1794 50  0000 C CNN
+F 2 "Connector_PinHeader_2.54mm:PinHeader_1x04_P2.54mm_Vertical" H 8500 1600 50  0001 C CNN
+F 3 "~" H 8500 1600 50  0001 C CNN
+	1    8500 1600
+	-1   0    0    -1
+$EndComp
+$Comp
+L power:VCC #PWR0104
+U 1 1 5E36750E
+P 7000 1500
+F 0 "#PWR0104" H 7000 1350 50  0001 C CNN
+F 1 "VCC" H 7017 1673 50  0000 C CNN
+F 2 "" H 7000 1500 50  0001 C CNN
+F 3 "" H 7000 1500 50  0001 C CNN
+	1    7000 1500
+	0    -1   -1   0
+$EndComp
+Wire Wire Line
+	7200 1500 7000 1500
+$Comp
+L power:GND #PWR0105
+U 1 1 5E369373
+P 7000 1800
+F 0 "#PWR0105" H 7000 1550 50  0001 C CNN
+F 1 "GND" H 7005 1627 50  0000 C CNN
+F 2 "" H 7000 1800 50  0001 C CNN
+F 3 "" H 7000 1800 50  0001 C CNN
+	1    7000 1800
+	0    1    1    0
+$EndComp
+Wire Wire Line
+	7200 1800 7000 1800
+$Comp
+L power:GND #PWR0106
+U 1 1 5E37858C
+P 9550 4300
+F 0 "#PWR0106" H 9550 4050 50  0001 C CNN
+F 1 "GND" H 9555 4127 50  0000 C CNN
+F 2 "" H 9550 4300 50  0001 C CNN
+F 3 "" H 9550 4300 50  0001 C CNN
+	1    9550 4300
+	-1   0    0    -1
+$EndComp
+Wire Wire Line
+	9550 4300 9550 3850
+$Comp
+L power:GND #PWR0107
+U 1 1 5E37C667
+P 9050 1800
+F 0 "#PWR0107" H 9050 1550 50  0001 C CNN
+F 1 "GND" H 9055 1627 50  0000 C CNN
+F 2 "" H 9050 1800 50  0001 C CNN
+F 3 "" H 9050 1800 50  0001 C CNN
+	1    9050 1800
+	0    -1   1    0
+$EndComp
+Wire Wire Line
+	8700 1800 9050 1800
+Wire Wire Line
+	8700 1500 9650 1500
+Wire Wire Line
+	9650 1500 9650 2250
+Wire Wire Line
+	9150 2950 9100 2950
+Wire Wire Line
+	9100 2950 9100 2050
+Wire Wire Line
+	9100 2050 9450 2050
+Wire Wire Line
+	9450 2050 9450 1600
+Wire Wire Line
+	9450 1600 8700 1600
+Wire Wire Line
+	9150 3050 9050 3050
+Wire Wire Line
+	9050 3050 9050 2000
+Wire Wire Line
+	9050 2000 9400 2000
+Wire Wire Line
+	9400 2000 9400 1700
+Wire Wire Line
+	9400 1700 8700 1700
+Wire Wire Line
+	5000 2650 5000 1600
+Wire Wire Line
+	5000 1600 7200 1600
+Wire Wire Line
+	5000 2750 5000 2700
+Wire Wire Line
+	5000 2700 6750 2700
+Wire Wire Line
+	6750 2700 6750 1700
+Wire Wire Line
+	6750 1700 7200 1700
+$Comp
+L power:GND #PWR0108
+U 1 1 5E39F09C
+P 9450 5150
+F 0 "#PWR0108" H 9450 4900 50  0001 C CNN
+F 1 "GND" H 9455 4977 50  0000 C CNN
+F 2 "" H 9450 5150 50  0001 C CNN
+F 3 "" H 9450 5150 50  0001 C CNN
+	1    9450 5150
+	0    -1   1    0
+$EndComp
+$Comp
+L power:VCC #PWR0109
+U 1 1 5E3A3B5B
+P 9450 4750
+F 0 "#PWR0109" H 9450 4600 50  0001 C CNN
+F 1 "VCC" H 9467 4923 50  0000 C CNN
+F 2 "" H 9450 4750 50  0001 C CNN
+F 3 "" H 9450 4750 50  0001 C CNN
+	1    9450 4750
+	0    1    1    0
+$EndComp
+$Comp
+L power:VCC #PWR0110
+U 1 1 5E3A5236
+P 9450 2150
+F 0 "#PWR0110" H 9450 2000 50  0001 C CNN
+F 1 "VCC" H 9467 2323 50  0000 C CNN
+F 2 "" H 9450 2150 50  0001 C CNN
+F 3 "" H 9450 2150 50  0001 C CNN
+	1    9450 2150
+	0    1    1    0
+$EndComp
+Wire Wire Line
+	9450 2150 9450 2250
+$Comp
+L Connector:Conn_01x05_Male J_USB1
+U 1 1 5E3B2E3A
+P 8500 4950
+F 0 "J_USB1" H 8608 5331 50  0000 C CNN
+F 1 "Conn_01x05_Male" H 8608 5240 50  0000 C CNN
+F 2 "Connector_PinHeader_2.54mm:PinHeader_1x05_P2.54mm_Vertical" H 8500 4950 50  0001 C CNN
+F 3 "~" H 8500 4950 50  0001 C CNN
+	1    8500 4950
+	1    0    0    -1
+$EndComp
+Wire Wire Line
+	8700 4750 9450 4750
+Wire Wire Line
+	8700 5150 9450 5150
 $EndSCHEMATC
